Commit message: replaced joint controllers with velocity controllers in rear

File: urdf/alt_car_assembly.urdf (robot description, URDF)
Before this commit: robot alt_car_assembly, 10 links, 9 joints
Joints:
- joint front_left_axle: limit effort=10 velocity=1 -> effort=100 velocity=10
- joint front_right_axle: limit effort=10 velocity=1 -> effort=100 velocity=10
- joint rear_left_axle: limit effort=10 velocity=1 -> effort=100 velocity=10
- joint rear_right_axle: limit effort=10 velocity=1 -> effort=100 velocity=10
